File: mc33063buck1.sch (KiCad schematic (older format))
At the start: 14 parts, among them Q1 MJE3055T, U1 MC34063

Commit message: make pcb layout.
Parts:
- added J1, J2, J3: Conn_01x01, Connectors:Pin_d1.3mm_L11.0mm, symbol Conn_01x01
- added J4: USB_A, Connectors:USB_A, symbol USB_A
- added J5: Jack-DC, Connectors:BARREL_JACK, symbol Jack-DC
- added R10, R8: 51k, Resistors_THT:R_Axial_DIN0309_L9.0mm_D3.2mm_P2.54mm_Vertical, symbol R
- added R6: 0.2, Resistors_THT:R_Bare_Metal_Element_L21.3mm_W4.8mm_P20.30mm, symbol R
- added R7: 43k, Resistors_THT:R_Axial_DIN0309_L9.0mm_D3.2mm_P2.54mm_Vertical, symbol R
- added R9: 75k, Resistors_THT:R_Axial_DIN0309_L9.0mm_D3.2mm_P2.54mm_Vertical, symbol R
- C1: footprint (none) -> Capacitors_THT:C_Disc_D11.0mm_W5.0mm_P5.00mm
- C2, C3: footprint (none) -> Capacitors_THT:CP_Radial_D12.5mm_P5.00mm
- D1: footprint (none) -> Diodes_THT:D_DO-201AD_P15.24mm_Horizontal
- D2: footprint (none) -> LEDs:LED_D5.0mm; symbol LED -> LED-RESCUE-mc33063buck1
- L1: footprint (none) -> Inductors_THT:L_Toroid_Vertical_L24.6mm_W15.5mm_P11.44mm_Pulse_KM-4
- Q1: footprint (none) -> TO_SOT_Packages_THT-2:TO-220_Neutral123_Vertical
- R1: footprint (none) -> Resistors_THT:R_Bare_Metal_Element_L21.3mm_W4.8mm_P20.30mm
- R2, R3, R4, R5: footprint (none) -> Resistors_THT:R_Axial_DIN0309_L9.0mm_D3.2mm_P2.54mm_Vertical
- RV1: footprint (none) -> Potentiometers:Potentiometer_Trimmer_ACP_CA6v_Horizontal; symbol POT -> POT-RESCUE-mc33063buck1
- U1: footprint (none) -> Housings_DIP:DIP-8_W7.62mm_LongPads
Connections:
- net Vout is gone; now on net +5V: C2.1, D2.2 (A), L1.2
- net GND: now also J2.1 (Pin_1), J4.4 (GND), J5.2, J5.3, R10.2, R8.2
- net at Q1.2 (C), R1.2, U1.1 (Sw_Coll)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: now also R6.2
- net +5V: now reaches R3.1
- net +5V: now also J3.1 (Pin_1), J4.1 (VBUS), R7.1, R9.1
- net Vin renamed +BATT
- net +BATT: now also J1.1 (Pin_1), J5.1, R6.1
- new net: J4.2 (D-), R7.2, R8.1
- new net: J4.3 (D+), R10.1, R9.2
- no-connect marks 0 -> 2
Other:
- moved on the sheet: C1, C2, C3, D1, D2, L1, Q1, R1, R2, R3, R4, R5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
